Commit message: Create visualization package. Fix related issues in description package.

File: lkwrbot_description/urdf/base.common.xacro (robot description, xacro)
@@ -31,5 +31,11 @@
   <xacro:property name="omniwheel_radius" value="${omniwheel_diameter/2}"/>
   <!-- Control related -->
-  <!-- TODO Determine if these should be spcified here or in a separate .urdf.xacro file -->
+  <!-- TODO Determine if these should be specified here or in a separate .urdf.xacro file -->
+  <!-- Configurable hardware parameters (STS3215 defaults) -->
+  <!-- HACK changed from arg to property-->
+  <xacro:property name="sts_max_velocity_steps" value="3400"/>  <!-- STS3215=3400, STS3032=2900, STS3235=3400 -->
+  <xacro:property name="proportional_acc_max"   value="25"/>    <!-- [0-254]; 0 = disable proportional ACC -->
+  <!-- Maximum allowable speed/acceleration/torque for each motor -->
+  <xacro:property name="max_velocity_steps" value="${int(sts_max_velocity_steps * 0.85)}"/> <!-- steps/second (85% of hardware max, 15% safety margin) -->
   <xacro:property name="max_velocity_rads" value="${max_velocity_steps*2*pi/4096}"/> <!-- rad/s -->
   <xacro:property name="max_torque_nm" value="2.942"/> <!-- N⋅m (30 kgf⋅cm for STS3215) -->

Commit message: Update dimensions and  mass

File: lkwrbot_description/urdf/base.common.xacro (robot description, xacro)
@@ -8,5 +8,5 @@
   <!-- Wheel mount offsets -->
   <xacro:property name="wheel_base_radius" value="0.132239"/> <!--TODO determine/measure correct value -->
-  <xacro:property name="wheel_base_offset_z" value="0.01036"/> <!--TODO determine/measure correct value -->
+  <xacro:property name="wheel_base_offset_z" value="0.010"/>
   <!-- 60° offset from X-axis -->
   <xacro:property name="wheel_radial_offset" value="${pi/3}"/>
@@ -23,10 +23,9 @@
   <xacro:property name="motormount_height" value="0.045"/>
   <xacro:property name="motormount_mass" value="0.010"/>
-  <xacro:property name="motormount_base_radius" value="${0.103 - motormount_depth/2}"/>
+  <xacro:property name="motormount_base_radius" value="${0.100 - motormount_depth/2}"/>
   <!-- Omniwheel dimensions-->
-  <!-- taken from datasheet/brochure -->
-  <xacro:property name="omniwheel_diameter" value="0.100"/>
-  <xacro:property name="omniwheel_width" value="0.030"/>
-  <xacro:property name="omniwheel_mass" value="0.290"/>
+  <xacro:property name="omniwheel_diameter" value="0.102"/>
+  <xacro:property name="omniwheel_width" value="0.031"/>
+  <xacro:property name="omniwheel_mass" value="0.292"/>  <!--incl. hub & bolts nuts -->
   <xacro:property name="omniwheel_radius" value="${omniwheel_diameter/2}"/>
   <!-- Control related -->
@@ -38,4 +37,6 @@
   <!-- Maximum allowable speed/acceleration/torque for each motor -->
   <xacro:property name="max_velocity_steps" value="${int(sts_max_velocity_steps * 0.85)}"/> <!-- steps/second (85% of hardware max, 15% safety margin) -->
+  <!-- VScode extension "Robot Developer Extensions for URDF" command 'URDF preview' can't handle int(...)-->
+  <!-- XXX xacro:property name="max_velocity_steps" value="$2890" --> <!-- steps/second (85% of hardware max, 15% safety margin) -->
   <xacro:property name="max_velocity_rads" value="${max_velocity_steps*2*pi/4096}"/> <!-- rad/s -->
   <xacro:property name="max_torque_nm" value="2.942"/> <!-- N⋅m (30 kgf⋅cm for STS3215) -->

File: lkwrbot_description/urdf/base.urdf.xacro (robot description, xacro)
@@ -7,5 +7,6 @@
   <link name="base_footprint"/>
   <xacro:lkwrbot_base_module parent="base_footprint">
-    <origin xyz="0 0 ${wheel_base_radius - wheel_base_offset_z}" rpy="0 0 0"/>
+    <origin xyz="0 0 ${omniwheel_radius - wheel_base_offset_z}" rpy="0 0 0"/>
+    <!-- XXX origin xyz="0 0 ${wheel_base_radius - wheel_base_offset_z}" rpy="0 0 0" -->
   </xacro:lkwrbot_base_module>
 </robot>

Commit message: Temp fix to prevent  a crash in the 'URDF Preview' command (from Robot Developer Extensions for URDF)

File: lkwrbot_description/urdf/base.common.xacro (robot description, xacro)
@@ -33,10 +33,10 @@
   <!-- Configurable hardware parameters (STS3215 defaults) -->
   <!-- HACK changed from arg to property-->
-  <xacro:property name="sts_max_velocity_steps" value="3400"/>  <!-- STS3215=3400, STS3032=2900, STS3235=3400 -->
-  <xacro:property name="proportional_acc_max"   value="25"/>    <!-- [0-254]; 0 = disable proportional ACC -->
+  <xacro:arg name="sts_max_velocity_steps" default="3400"/>  <!-- STS3215=3400, STS3032=2900, STS3235=3400 -->
+  <xacro:arg name="proportional_acc_max"   default="25"/>    <!-- [0-254]; 0 = disable proportional ACC -->
   <!-- Maximum allowable speed/acceleration/torque for each motor -->
-  <xacro:property name="max_velocity_steps" value="${int(sts_max_velocity_steps * 0.85)}"/> <!-- steps/second (85% of hardware max, 15% safety margin) -->
+  <!-- xacro:property name="max_velocity_steps" value="${int(sts_max_velocity_steps * 0.85)}" --> <!-- steps/second (85% of hardware max, 15% safety margin) -->
   <!-- VScode extension "Robot Developer Extensions for URDF" command 'URDF preview' can't handle int(...)-->
-  <!-- XXX xacro:property name="max_velocity_steps" value="$2890" --> <!-- steps/second (85% of hardware max, 15% safety margin) -->
+  <xacro:property name="max_velocity_steps" value="2890"/> <!-- steps/second (85% of hardware max, 15% safety margin) -->
   <xacro:property name="max_velocity_rads" value="${max_velocity_steps*2*pi/4096}"/> <!-- rad/s -->
   <xacro:property name="max_torque_nm" value="2.942"/> <!-- N⋅m (30 kgf⋅cm for STS3215) -->

File: lkwrbot_description/urdf/base.urdf.xacro (robot description, xacro)
@@ -8,5 +8,4 @@
   <xacro:lkwrbot_base_module parent="base_footprint">
     <origin xyz="0 0 ${omniwheel_radius - wheel_base_offset_z}" rpy="0 0 0"/>
-    <!-- XXX origin xyz="0 0 ${wheel_base_radius - wheel_base_offset_z}" rpy="0 0 0" -->
   </xacro:lkwrbot_base_module>
 </robot>

Commit message: Add serv-motorss

File: lkwrbot_description/urdf/base.common.xacro (robot description, xacro)
@@ -4,4 +4,5 @@
   <xacro:property name="white_smoke_rgba" value="0.961 0.961 0.961 1.0"/>
   <xacro:property name="dim_grey_rgba" value="0.412 0.412 0.412 1.0"/>
+  <xacro:property name="greyish_black_rgba" value="0.314 0.314 0.314 1.0"/>
   <!-- Base mesh rotation about Z (rad) -->
   <xacro:property name="base_offset_rz" value="${3*pi/2}"/> <!-- TODO check still used -->
@@ -10,7 +11,7 @@
   <xacro:property name="wheel_base_offset_z" value="0.010"/>
   <!-- 60° offset from X-axis -->
-  <xacro:property name="wheel_radial_offset" value="${pi/3}"/>
+  <xacro:property name="radial_offset" value="${pi/3}"/>
   <!-- 120° between wheels -->
-  <xacro:property name="wheel_radial_theta" value="${2*pi/3}"/>
+  <xacro:property name="radial_theta" value="${2*pi/3}"/>
   <!-- Plate dimensions-->
   <xacro:property name="base_plate_diameter" value="0.215"/>
@@ -23,5 +24,11 @@
   <xacro:property name="motormount_height" value="0.045"/>
   <xacro:property name="motormount_mass" value="0.010"/>
-  <xacro:property name="motormount_base_radius" value="${0.100 - motormount_depth/2}"/>
+  <xacro:property name="motormount_base_radius" value="${0.100 - motormount_depth/2}"/> <!--TODO determine/measure correct value -->
+  <!-- Servo dimensions-->
+  <xacro:property name="servo_depth" value="0.035"/>
+  <xacro:property name="servo_width" value="0.025"/>
+  <xacro:property name="servo_height" value="0.045"/>
+  <xacro:property name="servo_mass" value="0.054"/>
+   <xacro:property name="servo_base_radius" value="${0.100 - motormount_depth/2 - servo_depth/2 + 0.004}"/> <!--TODO determine/measure correct value -->
   <!-- Omniwheel dimensions-->
   <xacro:property name="omniwheel_diameter" value="0.102"/>

File: lkwrbot_description/urdf/base.module.xacro (robot description, xacro)
@@ -4,5 +4,5 @@
   <xacro:include filename="$(find lkwrbot_description)/urdf/base.common.xacro"/>
   <xacro:macro name="lkwrbot_base_module" params="parent *origin">
-    <!-- Material definitions -->
+    <!-- === Material definitions === -->
     <material name="base_material">
       <color rgba="${white_smoke_rgba}"/>
@@ -11,4 +11,7 @@
       <color rgba="${dim_grey_rgba}"/>
     </material>
+    <material name="servo_material">
+      <color rgba="${greyish_black_rgba}"/>
+    </material>
     <!-- Mount base_link to parent platform at specified origin -->
     <joint name="lkwrbot_mount_joint" type="fixed">
@@ -17,4 +20,5 @@
       <xacro:insert_block name="origin"/>
     </joint>
+    <!-- === Links === -->
     <!-- Bottom base plate -->
     <link name="bottom_base_plate_link">
@@ -51,5 +55,4 @@
       <xacro:inertial_cylinder mass="${top_base_plate_mass}" radius="${base_plate_diameter/2}" length="${base_plate_height}"/>
     </link>
-    <!-- TODO add servo's -->
     <!-- Left motor mount -->
     <link name="left_motormount_link">
@@ -88,4 +91,40 @@
       <xacro:default_inertial mass="${motormount_mass}"/>
     </link>
+    <!-- Left servo -->
+    <link name="left_servo_link">
+      <visual>
+        <origin xyz="${servo_depth/2} 0 ${servo_height/2}" rpy="0 ${pi/2} 0"/>
+        <geometry>
+          <mesh filename="package://lkwrbot_description/meshes/servomotor_STS3215.stl" scale="0.001 0.001 0.001"/>
+        </geometry>
+        <material name="servo_material"/>
+      </visual>
+      <!-- No collision element: inside robot -->
+      <xacro:default_inertial mass="${servo_mass}"/>
+    </link>
+    <!-- back servo -->
+    <link name="back_servo_link">
+      <visual>
+        <origin xyz="${servo_depth/2} 0 ${servo_height/2}" rpy="0 ${pi/2} 0"/>
+        <geometry>
+          <mesh filename="package://lkwrbot_description/meshes/servomotor_STS3215.stl" scale="0.001 0.001 0.001"/>
+        </geometry>
+        <material name="servo_material"/>
+      </visual>
+      <!-- No collision element: inside robot -->
+      <xacro:default_inertial mass="${servo_mass}"/>
+    </link>
+    <!-- Right servo -->
+    <link name="right_servo_link">
+      <visual>
+        <origin xyz="${servo_depth/2} 0 ${servo_height/2}" rpy="0 ${pi/2} 0"/>
+        <geometry>
+          <mesh filename="package://lkwrbot_description/meshes/servomotor_STS3215.stl" scale="0.001 0.001 0.001"/>
+        </geometry>
+        <material name="servo_material"/>
+      </visual>
+      <!-- No collision element: inside robot -->
+      <xacro:default_inertial mass="${servo_mass}"/>
+    </link>
     <!-- Left wheel -->
     <link name="left_wheel_link">
@@ -142,5 +181,5 @@
       <xacro:inertial_cylinder mass="${omniwheel_mass}" radius="${omniwheel_radius}" length="${omniwheel_width}"/>
     </link>
-    <!-- JOINTS -->
+    <!-- === Joints === -->
     <joint name="top_plate_joint" type="fixed">
       <parent link="bottom_base_plate_link"/>
@@ -152,5 +191,5 @@
       <parent link="bottom_base_plate_link"/>
       <child link="left_motormount_link"/>
-      <origin xyz="${motormount_base_radius * cos(wheel_radial_offset)} ${motormount_base_radius * sin(wheel_radial_offset)} 0" rpy="0 0 ${wheel_radial_offset}"/>
+      <origin xyz="${motormount_base_radius * cos(radial_offset)} ${motormount_base_radius * sin(radial_offset)} 0" rpy="0 0 ${radial_offset}"/>
     </joint>
     <!-- back motormount joint: 180 degrees anti-clockwise from +X at radius base_radius -->
@@ -158,5 +197,5 @@
       <parent link="bottom_base_plate_link"/>
       <child link="back_motormount_link"/>
-      <origin xyz="${motormount_base_radius * cos(wheel_radial_offset + wheel_radial_theta)} ${motormount_base_radius * sin(wheel_radial_offset + wheel_radial_theta)} 0" rpy="0 0 ${wheel_radial_offset + wheel_radial_theta}"/>
+      <origin xyz="${motormount_base_radius * cos(radial_offset + radial_theta)} ${motormount_base_radius * sin(radial_offset + radial_theta)} 0" rpy="0 0 ${radial_offset + radial_theta}"/>
     </joint>
     <!-- right motormount joint: 300 degrees (or -60 degrees) anti-clockwise from +X at radius base_radius -->
@@ -164,5 +203,23 @@
       <parent link="bottom_base_plate_link"/>
       <child link="right_motormount_link"/>
-      <origin xyz="${motormount_base_radius * cos(wheel_radial_offset - wheel_radial_theta)} ${motormount_base_radius * sin(wheel_radial_offset - wheel_radial_theta)} 0" rpy="0 0 ${wheel_radial_offset - wheel_radial_theta}"/>
+      <origin xyz="${motormount_base_radius * cos(radial_offset - radial_theta)} ${motormount_base_radius * sin(radial_offset - radial_theta)} 0" rpy="0 0 ${radial_offset - radial_theta}"/>
+    </joint>
+    <!-- left servo joint: 60 degrees anti-clockwise from +X at radius wheel_base_radius -->
+    <joint name="left_servo_joint" type="fixed">
+      <parent link="bottom_base_plate_link"/>
+      <child link="left_servo_link"/>
+      <origin xyz="${servo_base_radius * cos(radial_offset)} ${servo_base_radius * sin(radial_offset)} 0" rpy="0 0 ${radial_offset}"/>
+    </joint>
+    <!-- back servo joint: 180 degrees anti-clockwise from +X at radius base_radius -->
+   <joint name="back_servo_joint" type="fixed">
+      <parent link="bottom_base_plate_link"/>
+      <child link="back_servo_link"/>
+      <origin xyz="${servo_base_radius * cos(radial_offset + radial_theta)} ${servo_base_radius * sin(radial_offset + radial_theta)} 0" rpy="0 0 ${radial_offset + radial_theta}"/>
+    </joint>
+    <!-- right servo joint: 300 degrees (or -60 degrees) anti-clockwise from +X at radius base_radius -->
+    <joint name="right_servo_joint" type="fixed">
+      <parent link="bottom_base_plate_link"/>
+      <child link="right_servo_link"/>
+      <origin xyz="${servo_base_radius * cos(radial_offset - radial_theta)} ${servo_base_radius * sin(radial_offset - radial_theta)} 0" rpy="0 0 ${radial_offset - radial_theta}"/>
     </joint>
     <!-- left wheel joint: 60 degrees anti-clockwise from +X at radius wheel_base_radius -->
@@ -170,5 +227,5 @@
       <parent link="bottom_base_plate_link"/>
       <child link="left_wheel_link"/>
-      <origin xyz="${wheel_base_radius * cos(wheel_radial_offset)} ${wheel_base_radius * sin(wheel_radial_offset)} ${wheel_base_offset_z}" rpy="0 ${pi/2} ${wheel_radial_offset}"/>
+      <origin xyz="${wheel_base_radius * cos(radial_offset)} ${wheel_base_radius * sin(radial_offset)} ${wheel_base_offset_z}" rpy="0 ${pi/2} ${radial_offset}"/>
       <axis xyz="0 0 1"/>
       <limit effort="${max_torque_nm}" velocity="${max_velocity_rads}"/>
@@ -178,5 +235,5 @@
       <parent link="bottom_base_plate_link"/>
       <child link="back_wheel_link"/>
-      <origin xyz="${wheel_base_radius * cos(wheel_radial_offset + wheel_radial_theta)} ${wheel_base_radius * sin(wheel_radial_offset + wheel_radial_theta)} ${wheel_base_offset_z}" rpy="0 ${pi/2} ${wheel_radial_offset + wheel_radial_theta}"/>
+      <origin xyz="${wheel_base_radius * cos(radial_offset + radial_theta)} ${wheel_base_radius * sin(radial_offset + radial_theta)} ${wheel_base_offset_z}" rpy="0 ${pi/2} ${radial_offset + radial_theta}"/>
       <axis xyz="0 0 1"/>
       <limit effort="${max_torque_nm}" velocity="${max_velocity_rads}" />
@@ -186,5 +243,5 @@
       <parent link="bottom_base_plate_link"/>
       <child link="right_wheel_link"/>
-      <origin xyz="${wheel_base_radius * cos(wheel_radial_offset - wheel_radial_theta)} ${wheel_base_radius * sin(wheel_radial_offset - wheel_radial_theta)} ${wheel_base_offset_z}" rpy="0 ${pi/2} ${wheel_radial_offset - wheel_radial_theta}"/>
+      <origin xyz="${wheel_base_radius * cos(radial_offset - radial_theta)} ${wheel_base_radius * sin(radial_offset - radial_theta)} ${wheel_base_offset_z}" rpy="0 ${pi/2} ${radial_offset - radial_theta}"/>
       <axis xyz="0 0 1"/>
       <limit effort="${max_torque_nm}" velocity="${max_velocity_rads}" />

Commit message: Add (empty) control.xacro.

File: lkwrbot_description/urdf/base.common.xacro (robot description, xacro)
@@ -30,5 +30,5 @@
   <xacro:property name="servo_height" value="0.045"/>
   <xacro:property name="servo_mass" value="0.054"/>
-   <xacro:property name="servo_base_radius" value="${0.100 - motormount_depth/2 - servo_depth/2 + 0.004}"/> <!--TODO determine/measure correct value -->
+  <xacro:property name="servo_base_radius" value="${0.100 - motormount_depth/2 - servo_depth/2 + 0.004}"/> <!--TODO determine/measure correct value -->
   <!-- Omniwheel dimensions-->
   <xacro:property name="omniwheel_diameter" value="0.102"/>

File: lkwrbot_description/urdf/base.module.xacro (robot description, xacro)
@@ -3,4 +3,5 @@
   <xacro:include filename="$(find lkwrbot_description)/urdf/inertia_tensors.urdf.xacro"/>
   <xacro:include filename="$(find lkwrbot_description)/urdf/base.common.xacro"/>
+  <xacro:include filename="$(find lkwrbot_description)/urdf/base.control.xacro"/>
   <xacro:macro name="lkwrbot_base_module" params="parent *origin">
     <!-- === Material definitions === -->
