Commit message: Initial commit for control package and  (related) changed  urdf.xacro files in description package.

File: lkwrbot_description/urdf/base.common.xacro (robot description, xacro)
@@ -1,17 +1,11 @@
 <?xml version="1.0"?>
 <robot xmlns:xacro="http://www.ros.org/wiki/xacro">
-  <!-- Colors (RGBA) -->
-  <xacro:property name="white_smoke_rgba" value="0.961 0.961 0.961 1.0"/>
-  <xacro:property name="dim_grey_rgba" value="0.412 0.412 0.412 1.0"/>
-  <xacro:property name="greyish_black_rgba" value="0.314 0.314 0.314 1.0"/>
-  <!-- Base mesh rotation about Z (rad) -->
-  <xacro:property name="base_offset_rz" value="${3*pi/2}"/> <!-- TODO check still used -->
+  <!-- Common dimensions for the base of the LKWrbot robot -->
   <!-- Wheel mount offsets -->
   <xacro:property name="wheel_base_radius" value="0.132239"/> <!--TODO determine/measure correct value -->
   <xacro:property name="wheel_base_offset_z" value="0.010"/>
-  <!-- 60° offset from X-axis -->
-  <xacro:property name="radial_offset" value="${pi/3}"/>
-  <!-- 120° between wheels -->
-  <xacro:property name="radial_theta" value="${2*pi/3}"/>
+  <!-- three-wheel-drive radial offsets -->
+  <xacro:property name="radial_offset" value="${pi/3}"/> <!-- 60° offset from X-axis -->
+  <xacro:property name="radial_theta" value="${2*pi/3}"/> <!-- 120° between wheels -->
   <!-- Plate dimensions-->
   <xacro:property name="base_plate_diameter" value="0.215"/>
@@ -36,15 +30,3 @@
   <xacro:property name="omniwheel_mass" value="0.292"/>  <!--incl. hub & bolts nuts -->
   <xacro:property name="omniwheel_radius" value="${omniwheel_diameter/2}"/>
-  <!-- Control related -->
-  <!-- TODO Determine if these should be specified here or in a separate .urdf.xacro file -->
-  <!-- Configurable hardware parameters (STS3215 defaults) -->
-  <!-- HACK changed from arg to property-->
-  <xacro:arg name="sts_max_velocity_steps" default="3400"/>  <!-- STS3215=3400, STS3032=2900, STS3235=3400 -->
-  <xacro:arg name="proportional_acc_max"   default="25"/>    <!-- [0-254]; 0 = disable proportional ACC -->
-  <!-- Maximum allowable speed/acceleration/torque for each motor -->
-  <!-- xacro:property name="max_velocity_steps" value="${int(sts_max_velocity_steps * 0.85)}" --> <!-- steps/second (85% of hardware max, 15% safety margin) -->
-  <!-- VScode extension "Robot Developer Extensions for URDF" command 'URDF preview' can't handle int(...)-->
-  <xacro:property name="max_velocity_steps" value="2890"/> <!-- steps/second (85% of hardware max, 15% safety margin) -->
-  <xacro:property name="max_velocity_rads" value="${max_velocity_steps*2*pi/4096}"/> <!-- rad/s -->
-  <xacro:property name="max_torque_nm" value="2.942"/> <!-- N⋅m (30 kgf⋅cm for STS3215) -->
 </robot>

File: lkwrbot_description/urdf/base.control.xacro (robot description, xacro)
@@ -1,3 +1,89 @@
 <?xml version="1.0"?>
 <robot xmlns:xacro="http://www.ros.org/wiki/xacro">
+<!-- Arguments (externally settable via command line or parent xacro) -->
+  <xacro:arg name="serial_port" default="/dev/ttySERVO"/>
+  <xacro:arg name="baud_rate" default="1000000"/>
+  <xacro:arg name="use_mock" default="false"/>
+  <xacro:arg name="use_sync_write" default="true"/>
+  <xacro:arg name="left_motor_id" default="7"/>
+  <xacro:arg name="back_motor_id" default="8"/>
+  <xacro:arg name="right_motor_id" default="9"/>
+  <!-- Configurable hardware parameters (STS3215 defaults) -->
+  <xacro:arg name="sts_max_velocity_steps" default="3400"/>  <!-- STS3215=3400, STS3032=2900, STS3235=3400 -->
+  <xacro:arg name="proportional_acc_max"   default="25"/>    <!-- [0-254]; 0 = disable proportional ACC -->
+  <!-- Base operating mode -->
+  <xacro:property name="base_operating_mode" value="1"/>  <!-- Velocity mode -->
+  <!-- Motor-specific parameter — sourced from arg, STS3215 default -->
+  <xacro:property name="sts_max_velocity_steps" value="$(arg sts_max_velocity_steps)"/>  <!-- Max hardware velocity in steps/s -->
+  <!-- Proportional ACC parameters (SyncWriteSpe velocity path only) -->
+  <!-- ACC given to the wheel with the largest |target - current| velocity delta. -->
+  <!-- All others scaled proportionally so every wheel finishes ramping in equal time. -->
+  <!-- Set proportional_acc_max to 0 to disable (ACC=0 for all wheels). -->
+  <xacro:property name="proportional_acc_max" value="$(arg proportional_acc_max)"/>        <!-- [0-254] -->
+  <!-- Maximum allowable speed/acceleration/torque for each motor -->
+  <!-- Note: max_velocity_rads and max_torque_nm are used in <limit> in the base.module.xacro -->
+  <xacro:property name="max_velocity_steps" value="${int(sts_max_velocity_steps * 0.85)}"/> <!-- steps/second (85% of hardware max, 15% safety margin) -->
+  <xacro:property name="max_velocity_rads" value="${max_velocity_steps*2*pi/4096}"/> <!-- rad/s -->
+  <xacro:property name="max_torque_nm" value="2.942"/> <!-- N⋅m (30 kgf⋅cm for STS3215) -->
+  <!-- Omnidirectional Kinematics Calculations -->
+  <!-- For 3-wheel omni drive: ω_i = (-sin(θ_i)·v_x + cos(θ_i)·v_y + R·ω_z) / r -->
+  <!-- Maximum allowable linear velocity per axis -->
+  <xacro:property name="max_linear_velocity_x"  value="${omniwheel_radius * max_velocity_rads / (sqrt(3)/2)}"/>
+  <xacro:property name="max_linear_velocity_y"  value="${omniwheel_radius * max_velocity_rads / 1.0}"/>
+  <xacro:property name="max_angular_velocity_z" value="${omniwheel_radius * max_velocity_rads / wheel_base_radius}"/>
+  <!-- ROS 2 CONTROL -->
+  <!-- System interface -->
+  <ros2_control name="lkwrbot_base" type="system">
+    <hardware>
+      <plugin>sts_hardware_interface/STSHardwareInterface</plugin>
+      <!-- Serial communication parameters -->
+      <param name="serial_port">$(arg serial_port)</param>
+      <param name="baud_rate">$(arg baud_rate)</param>
+      <param name="use_sync_write">$(arg use_sync_write)</param>
+      <param name="enable_mock_mode">$(arg use_mock)</param>
+      <!-- Motor-specific parameter (adjust for different STS motor models) -->
+      <param name="max_velocity_steps">${sts_max_velocity_steps}</param>
+      <!-- Proportional ACC: scale per-wheel acceleration so all wheels finish ramping in equal time -->
+      <param name="proportional_acc_max">${proportional_acc_max}</param>
+    </hardware>
+    <!-- Left wheel joint (Motor ID 7) -->
+    <joint name="left_wheel_joint">
+      <param name="motor_id">$(arg left_motor_id)</param>
+      <param name="operating_mode">${base_operating_mode}</param>
+      <command_interface name="velocity"/>
+      <state_interface name="position"/>
+      <state_interface name="velocity"/>
+      <state_interface name="effort"/>
+      <state_interface name="voltage"/>
+      <state_interface name="temperature"/>
+      <state_interface name="current"/>
+      <state_interface name="is_moving"/>
+    </joint>
+    <!-- Back wheel joint (Motor ID 8) -->
+    <joint name="back_wheel_joint">
+      <param name="motor_id">$(arg back_motor_id)</param>
+      <param name="operating_mode">${base_operating_mode}</param>
+      <command_interface name="velocity"/>
+      <state_interface name="position"/>
+      <state_interface name="velocity"/>
+      <state_interface name="effort"/>
+      <state_interface name="voltage"/>
+      <state_interface name="temperature"/>
+      <state_interface name="current"/>
+      <state_interface name="is_moving"/>
+    </joint>
+    <!-- Right wheel joint (Motor ID 9) -->
+    <joint name="right_wheel_joint">
+      <param name="motor_id">$(arg right_motor_id)</param>
+      <param name="operating_mode">${base_operating_mode}</param>
+      <command_interface name="velocity"/>
+      <state_interface name="position"/>
+      <state_interface name="velocity"/>
+      <state_interface name="effort"/>
+      <state_interface name="voltage"/>
+      <state_interface name="temperature"/>
+      <state_interface name="current"/>
+      <state_interface name="is_moving"/>
+    </joint>
+  </ros2_control>
 </robot>

File: lkwrbot_description/urdf/base.module.xacro (robot description, xacro)
@@ -2,17 +2,7 @@
 <robot xmlns:xacro="http://www.ros.org/wiki/xacro">
   <xacro:include filename="$(find lkwrbot_description)/urdf/inertia_tensors.urdf.xacro"/>
-  <xacro:include filename="$(find lkwrbot_description)/urdf/base.common.xacro"/>
-  <xacro:include filename="$(find lkwrbot_description)/urdf/base.control.xacro"/>
+  <!-- xacro:include filename="$(find lkwrbot_description)/urdf/base.control.xacro"  TODO remove, now in base.urdf.xacro -->
   <xacro:macro name="lkwrbot_base_module" params="parent *origin">
-    <!-- === Material definitions === -->
-    <material name="base_material">
-      <color rgba="${white_smoke_rgba}"/>
-    </material>
-    <material name="omniwheel_material">
-      <color rgba="${dim_grey_rgba}"/>
-    </material>
-    <material name="servo_material">
-      <color rgba="${greyish_black_rgba}"/>
-    </material>
+    <xacro:include filename="$(find lkwrbot_description)/urdf/base.materials.xacro"/>
     <!-- Mount base_link to parent platform at specified origin -->
     <joint name="lkwrbot_mount_joint" type="fixed">
@@ -238,5 +228,5 @@
       <origin xyz="${wheel_base_radius * cos(radial_offset + radial_theta)} ${wheel_base_radius * sin(radial_offset + radial_theta)} ${wheel_base_offset_z}" rpy="0 ${pi/2} ${radial_offset + radial_theta}"/>
       <axis xyz="0 0 1"/>
-      <limit effort="${max_torque_nm}" velocity="${max_velocity_rads}" />
+      <limit effort="${max_torque_nm}" velocity="${max_velocity_rads}"/>
     </joint>
     <!-- right wheel joint: 300 degrees (or -60 degrees) anti-clockwise from +X at radius base_radius -->
@@ -246,5 +236,5 @@
       <origin xyz="${wheel_base_radius * cos(radial_offset - radial_theta)} ${wheel_base_radius * sin(radial_offset - radial_theta)} ${wheel_base_offset_z}" rpy="0 ${pi/2} ${radial_offset - radial_theta}"/>
       <axis xyz="0 0 1"/>
-      <limit effort="${max_torque_nm}" velocity="${max_velocity_rads}" />
+      <limit effort="${max_torque_nm}" velocity="${max_velocity_rads}"/>
     </joint>
   </xacro:macro>

File: lkwrbot_description/urdf/base.urdf.xacro (robot description, xacro)
@@ -3,5 +3,5 @@
   <xacro:include filename="$(find lkwrbot_description)/urdf/base.common.xacro"/>
   <xacro:include filename="$(find lkwrbot_description)/urdf/base.module.xacro"/>
-  <!-- xacro:include filename="$(find lkwrbot_description)/urdf/base.control.xacro" -->
+  <xacro:include filename="$(find lkwrbot_description)/urdf/base.control.xacro"/>
   <!-- Standalone lkwrbot base -->
   <link name="base_footprint"/>

Commit message: Update robot dimensions, enable  use-mock

File: lkwrbot_description/urdf/base.common.xacro (robot description, xacro)
@@ -3,6 +3,9 @@
   <!-- Common dimensions for the base of the LKWrbot robot -->
   <!-- Wheel mount offsets -->
-  <xacro:property name="wheel_base_radius" value="0.132239"/> <!--TODO determine/measure correct value -->
+  <xacro:property name="wheel_base_radius" value="0.134"/>  <!-- Calculated distance (from several measurements) -->
   <xacro:property name="wheel_base_offset_z" value="0.010"/>
+  <!--Measured distances -->
+  <xacro:property name="motormount_backside_radius" value="0.069"/> <!-- Distance from plate centre to back of motormount -->
+  <xacro:property name="motormount_servo_offset" value="0.004"/>  <!-- Offset distance back motormount to back of servo -->
   <!-- three-wheel-drive radial offsets -->
   <xacro:property name="radial_offset" value="${pi/3}"/> <!-- 60° offset from X-axis -->
@@ -18,5 +21,5 @@
   <xacro:property name="motormount_height" value="0.045"/>
   <xacro:property name="motormount_mass" value="0.010"/>
-  <xacro:property name="motormount_base_radius" value="${0.100 - motormount_depth/2}"/> <!--TODO determine/measure correct value -->
+  <xacro:property name="motormount_base_radius" value="${motormount_backside_radius + motormount_depth/2}"/>
   <!-- Servo dimensions-->
   <xacro:property name="servo_depth" value="0.035"/>
@@ -24,5 +27,5 @@
   <xacro:property name="servo_height" value="0.045"/>
   <xacro:property name="servo_mass" value="0.054"/>
-  <xacro:property name="servo_base_radius" value="${0.100 - motormount_depth/2 - servo_depth/2 + 0.004}"/> <!--TODO determine/measure correct value -->
+  <xacro:property name="servo_base_radius" value="${motormount_backside_radius + motormount_servo_offset + servo_depth/2 }"/>
   <!-- Omniwheel dimensions-->
   <xacro:property name="omniwheel_diameter" value="0.102"/>
