Commit message: Add servowheelhib to urdf.xacro's

File: lkwrbot_description/urdf/base.common.xacro (robot description, xacro)
@@ -28,7 +28,13 @@
   <xacro:property name="servo_mass" value="0.054"/>
   <xacro:property name="servo_base_radius" value="${motormount_backside_radius + motormount_servo_offset + servo_depth/2 }"/>
+  <!-- Servowheel hub dimensions-->
+  <xacro:property name="servowheelhub_diameter" value="0.030"/>
+  <xacro:property name="servowheelhub_width" value="0.014"/>
+  <xacro:property name="servowheelhub_mass" value="0.009"/>
+  <xacro:property name="servowheelhub_radius" value="${servowheelhub_diameter/2}"/>
   <!-- Omniwheel dimensions-->
   <xacro:property name="omniwheel_diameter" value="0.102"/>
-  <xacro:property name="omniwheel_width" value="0.031"/>
+  <xacro:property name="omniwheel_width" value="0.037"/>  <!-- Overall width incl rollers -->
+  <xacro:property name="omniwheel_hub_width" value="0.034"/> <!-- Width around the hub -->
   <xacro:property name="omniwheel_mass" value="0.292"/>  <!--incl. hub & bolts nuts -->
   <xacro:property name="omniwheel_radius" value="${omniwheel_diameter/2}"/>

File: lkwrbot_description/urdf/base.module.xacro (robot description, xacro)
@@ -118,4 +118,42 @@
       <xacro:default_inertial mass="${servo_mass}"/>
     </link>
+    <!-- left servowheelhub -->
+    <link name="left_servowheelhub_link">
+      <visual>
+        <origin xyz="0 0 -${omniwheel_hub_width/2}" rpy="0 0 0"/>
+        <geometry>
+          <mesh filename="package://lkwrbot_description/meshes/servowheelhub.stl" scale="0.001 0.001 0.001"/>
+        </geometry>
+        <material name="base_material"/>
+      </visual>
+      <!-- No collision element: inside robot -->
+      <!-- Assuming inertia is comparable to a cylinder (flange is excluded) -->
+      <xacro:inertial_cylinder mass="${servowheelhub_mass}" radius="${servowheelhub_radius}" length="${servowheelhub_width}"/>
+    </link>
+    <link name="back_servowheelhub_link">
+      <visual>
+        <origin xyz="0 0 -${omniwheel_hub_width/2}" rpy="0 0 0"/>
+        <geometry>
+          <mesh filename="package://lkwrbot_description/meshes/servowheelhub.stl" scale="0.001 0.001 0.001"/>
+        </geometry>
+        <material name="base_material"/>
+      </visual>
+      <!-- No collision element: inside robot -->
+      <!-- Assuming inertia is comparable to a cylinder (flange is excluded) -->
+      <xacro:inertial_cylinder mass="${servowheelhub_mass}" radius="${servowheelhub_radius}" length="${servowheelhub_width}"/>
+    </link>
+    <!-- right servowheelhub -->
+    <link name="right_servowheelhub_link">
+      <visual>
+        <origin xyz="0 0 -${omniwheel_hub_width/2}" rpy="0 0 0"/>
+        <geometry>
+          <mesh filename="package://lkwrbot_description/meshes/servowheelhub.stl" scale="0.001 0.001 0.001"/>
+        </geometry>
+        <material name="base_material"/>
+      </visual>
+      <!-- No collision element: inside robot -->
+      <!-- Assuming inertia is comparable to a cylinder (flange is excluded) -->
+      <xacro:inertial_cylinder mass="${servowheelhub_mass}" radius="${servowheelhub_radius}" length="${servowheelhub_width}"/>
+    </link>
     <!-- Left wheel -->
     <link name="left_wheel_link">
@@ -222,4 +260,10 @@
       <limit effort="${max_torque_nm}" velocity="${max_velocity_rads}"/>
     </joint>
+    <!-- left servowheelhub joint -->
+    <joint name="left_servowheelhub_joint" type="fixed">
+      <parent link="left_wheel_link"/>
+      <child link="left_servowheelhub_link"/>
+      <origin xyz="0 0 0" rpy="0 0 0"/>
+    </joint>
     <!-- back wheel joint: 180 degrees anti-clockwise from +X at radius base_radius -->
     <joint name="back_wheel_joint" type="continuous">
@@ -230,4 +274,10 @@
       <limit effort="${max_torque_nm}" velocity="${max_velocity_rads}"/>
     </joint>
+    <!-- back servowheelhub joint -->
+    <joint name="back_servowheelhub_joint" type="fixed">
+      <parent link="back_wheel_link"/>
+      <child link="back_servowheelhub_link"/>
+      <origin xyz="0 0 0" rpy="0 0 0"/>
+    </joint>
     <!-- right wheel joint: 300 degrees (or -60 degrees) anti-clockwise from +X at radius base_radius -->
     <joint name="right_wheel_joint" type="continuous">
@@ -238,4 +288,10 @@
       <limit effort="${max_torque_nm}" velocity="${max_velocity_rads}"/>
     </joint>
+    <!-- right servowheelhub joint -->
+    <joint name="right_servowheelhub_joint" type="fixed">
+      <parent link="right_wheel_link"/>
+      <child link="right_servowheelhub_link"/>
+      <origin xyz="0 0 0" rpy="0 0 0"/>
+    </joint>
   </xacro:macro>
 </robot>

Commit message: Update  dimensions, cleanup and format xacro's

File: lkwrbot_description/urdf/base.common.xacro (robot description, xacro)
@@ -3,9 +3,9 @@
   <!-- Common dimensions for the base of the LKWrbot robot -->
   <!-- Wheel mount offsets -->
-  <xacro:property name="wheel_base_radius" value="0.134"/>  <!-- Calculated distance (from several measurements) -->
+  <xacro:property name="wheel_base_radius" value="0.132"/>  <!-- Measured distance -->
   <xacro:property name="wheel_base_offset_z" value="0.010"/>
   <!--Measured distances -->
   <xacro:property name="motormount_backside_radius" value="0.069"/> <!-- Distance from plate centre to back of motormount -->
-  <xacro:property name="motormount_servo_offset" value="0.004"/>  <!-- Offset distance back motormount to back of servo -->
+  <xacro:property name="motormount_servo_offset" value="0.005"/>  <!-- Offset distance back motormount to back of servo -->
   <!-- three-wheel-drive radial offsets -->
   <xacro:property name="radial_offset" value="${pi/3}"/> <!-- 60° offset from X-axis -->

File: lkwrbot_description/urdf/base.control.xacro (robot description, xacro)
@@ -1,5 +1,5 @@
 <?xml version="1.0"?>
 <robot xmlns:xacro="http://www.ros.org/wiki/xacro">
-<!-- Arguments (externally settable via command line or parent xacro) -->
+  <!-- Arguments (externally settable via command line or parent xacro) -->
   <xacro:arg name="serial_port" default="/dev/ttySERVO"/>
   <xacro:arg name="baud_rate" default="1000000"/>

File: lkwrbot_description/urdf/base.module.xacro (robot description, xacro)
@@ -2,5 +2,4 @@
 <robot xmlns:xacro="http://www.ros.org/wiki/xacro">
   <xacro:include filename="$(find lkwrbot_description)/urdf/inertia_tensors.urdf.xacro"/>
-  <!-- xacro:include filename="$(find lkwrbot_description)/urdf/base.control.xacro"  TODO remove, now in base.urdf.xacro -->
   <xacro:macro name="lkwrbot_base_module" params="parent *origin">
     <xacro:include filename="$(find lkwrbot_description)/urdf/base.materials.xacro"/>
@@ -131,4 +130,5 @@
       <xacro:inertial_cylinder mass="${servowheelhub_mass}" radius="${servowheelhub_radius}" length="${servowheelhub_width}"/>
     </link>
+    <!-- back servowheelhub -->
     <link name="back_servowheelhub_link">
       <visual>

File: lkwrbot_description/urdf/inertia_tensors.urdf.xacro (robot description, xacro)
@@ -56,5 +56,5 @@
     </inertial>
   </xacro:macro>
-    <xacro:macro name="inertial_hollow_sphere_with_pose" params="mass diameter *origin">
+  <xacro:macro name="inertial_hollow_sphere_with_pose" params="mass diameter *origin">
     <inertial>
       <!-- Hollow sphere with pose-->
@@ -114,4 +114,4 @@
                                       izz="1e-3" />
     </inertial>
-</xacro:macro>
+  </xacro:macro>
 </robot>
