Commit message: Fix x-origin servo_link's

File: lkwrbot_description/urdf/base.module.xacro (robot description, xacro)
@@ -85,5 +85,5 @@
     <link name="left_servo_link">
       <visual>
-        <origin xyz="${servo_depth/2} 0 ${servo_height/2}" rpy="0 ${pi/2} 0"/>
+        <origin xyz="0 0 ${servo_height/2}" rpy="0 ${pi/2} 0"/>
         <geometry>
           <mesh filename="package://lkwrbot_description/meshes/servomotor_STS3215.stl" scale="0.001 0.001 0.001"/>
@@ -97,5 +97,5 @@
     <link name="back_servo_link">
       <visual>
-        <origin xyz="${servo_depth/2} 0 ${servo_height/2}" rpy="0 ${pi/2} 0"/>
+        <origin xyz="0 0 ${servo_height/2}" rpy="0 ${pi/2} 0"/>
         <geometry>
           <mesh filename="package://lkwrbot_description/meshes/servomotor_STS3215.stl" scale="0.001 0.001 0.001"/>
@@ -109,5 +109,5 @@
     <link name="right_servo_link">
       <visual>
-        <origin xyz="${servo_depth/2} 0 ${servo_height/2}" rpy="0 ${pi/2} 0"/>
+        <origin xyz="0 0 ${servo_height/2}" rpy="0 ${pi/2} 0"/>
         <geometry>
           <mesh filename="package://lkwrbot_description/meshes/servomotor_STS3215.stl" scale="0.001 0.001 0.001"/>
